File: var_state_eq/schematics/rev01/var_state_eq.brd (EAGLE design)
At the start: 74.6 x 59.7 mm, 69 parts, among them IC1 TL084P, IC2 TL084P, IC3 TL084P, J1 IN, J2 OUT

Commit message: Updates for part purchase
Parts:
- R26: value 22R -> 100R
- R31, R35: value 50K -> 56K
Changed lines of the file:
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@@
 <?xml version="1.0" encoding="utf-8"?>
 <!DOCTYPE eagle SYSTEM "eagle.dtd">
-<eagle version="9.6.1">
+<eagle version="9.5.1">
 <drawing>
 <settings>
@@
 <attribute name="VALUE" x="26.924" y="26.1112" size="1.27" layer="27" ratio="10"/>
 </element>
-<element name="R26" library="_common" package="0207/7" value="22R" x="49.53" y="21.59" smashed="yes" rot="R90">
+<element name="R26" library="_common" package="0207/7" value="100R" x="49.53" y="21.59" smashed="yes" rot="R90">
 <attribute name="NAME" x="50.165" y="19.558" size="1.27" layer="25" ratio="10" rot="R90"/>
 <attribute name="VALUE" x="50.0888" y="19.304" size="1.27" layer="27" ratio="10" rot="R90"/>
@@
 <attribute name="VALUE" x="5.715" y="13.335" size="1.27" layer="27" rot="R270"/>
 </element>
-<element name="R31" library="_common" package="0207/7" value="50K" x="19.05" y="29.21" smashed="yes">
+<element name="R31" library="_common" package="0207/7" value="56K" x="19.05" y="29.21" smashed="yes">
 <attribute name="NAME" x="17.653" y="28.702" size="1.27" layer="25" ratio="10"/>
 <attribute name="VALUE" x="16.764" y="28.6512" size="1.27" layer="27" ratio="10"/>
@@
 <attribute name="VALUE" x="31.496" y="3.0988" size="1.27" layer="27" ratio="10" rot="R180"/>
 </element>
-<element name="R35" library="_common" package="0207/7" value="50K" x="17.78" y="2.54" smashed="yes">
+<element name="R35" library="_common" package="0207/7" value="56K" x="17.78" y="2.54" smashed="yes">
 <attribute name="NAME" x="16.129" y="1.778" size="1.27" layer="25" ratio="10"/>
 <attribute name="VALUE" x="15.494" y="1.9812" size="1.27" layer="27" ratio="10"/>

Commit message: Updated resistor values to 56K
Parts:
- R21, R32: value 50K -> 56K
Changed lines of the file:
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@@
 <?xml version="1.0" encoding="utf-8"?>
 <!DOCTYPE eagle SYSTEM "eagle.dtd">
-<eagle version="9.5.1">
+<eagle version="9.5.2">
 <drawing>
 <settings>
@@
 <grid distance="50" unitdist="mil" unit="mm" style="lines" multiple="1" display="no" altdistance="5" altunitdist="mil" altunit="mm"/>
 <layers>
-<layer number="1" name="Top" color="4" fill="1" visible="yes" active="yes"/>
-<layer number="16" name="Bottom" color="1" fill="1" visible="yes" active="yes"/>
+<layer number="1" name="Top" color="4" fill="1" visible="no" active="yes"/>
+<layer number="16" name="Bottom" color="1" fill="1" visible="no" active="yes"/>
 <layer number="17" name="Pads" color="2" fill="1" visible="yes" active="yes"/>
 <layer number="18" name="Vias" color="2" fill="1" visible="yes" active="yes"/>
@@
 <attribute name="VALUE" x="5.715" y="55.245" size="1.27" layer="27" rot="R270"/>
 </element>
-<element name="R21" library="_common" package="0207/7" value="50K" x="20.32" y="53.34" smashed="yes">
+<element name="R21" library="_common" package="0207/7" value="56K" x="20.32" y="53.34" smashed="yes">
 <attribute name="NAME" x="18.923" y="52.705" size="1.27" layer="25" ratio="10"/>
 <attribute name="VALUE" x="18.034" y="52.7812" size="1.27" layer="27" ratio="10"/>
@@
 <attribute name="VALUE" x="16.764" y="28.6512" size="1.27" layer="27" ratio="10"/>
 </element>
-<element name="R32" library="_common" package="0207/7" value="50K" x="13.97" y="43.18" smashed="yes" rot="R270">
+<element name="R32" library="_common" package="0207/7" value="56K" x="13.97" y="43.18" smashed="yes" rot="R270">
 <attribute name="NAME" x="13.589" y="44.577" size="1.27" layer="25" ratio="10" rot="R270"/>
 <attribute name="VALUE" x="13.4112" y="45.466" size="1.27" layer="27" ratio="10" rot="R270"/>

Commit message: Updated cap values
Parts:
- C17, C9: value 100n -> 0.1uF
Changed lines of the file:
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@@
 <attribute name="VALUE" x="30.48" y="20.701" size="1.27" layer="27" ratio="10"/>
 </element>
-<element name="C17" library="_common" package="C025-024X044" value="100n" x="40.64" y="20.32" smashed="yes" rot="R180">
+<element name="C17" library="_common" package="C025-024X044" value="0.1uF" x="40.64" y="20.32" smashed="yes" rot="R180">
 <attribute name="NAME" x="42.418" y="18.923" size="1.27" layer="25" ratio="10" rot="R180"/>
 <attribute name="VALUE" x="42.418" y="22.987" size="1.27" layer="27" ratio="10" rot="R180"/>
@@
 <attribute name="VALUE" x="66.0654" y="45.2374" size="1.27" layer="27" ratio="10"/>
 </element>
-<element name="C9" library="_common" package="C025-024X044" value="100n" x="44.45" y="41.91" smashed="yes">
+<element name="C9" library="_common" package="C025-024X044" value="0.1uF" x="44.45" y="41.91" smashed="yes">
 <attribute name="NAME" x="44.577" y="43.307" size="1.27" layer="25" ratio="10"/>
 <attribute name="VALUE" x="42.672" y="39.243" size="1.27" layer="27" ratio="10"/>
